Commit message: feat: add depth camera to both sim & real dev

File: src/OrbbecSDK/orbbec_description/urdf/astra2.urdf.xacro (robot description, xacro)
@@ -86,5 +86,5 @@
   </link>
   <joint
-    name="camera_bottom_screw_joint"
+    name="camera_bottom_screw_frame"
     type="fixed">
     <origin
@@ -139,5 +139,5 @@
   </link>
   <joint
-    name="camera_ir_joint"
+    name="camera_ir_frame"
     type="fixed">
     <origin
@@ -192,5 +192,5 @@
   </link>
   <joint
-    name="camera_ir_optical_joint"
+    name="camera_ir_optical_frame"
     type="fixed">
     <origin
@@ -245,5 +245,5 @@
   </link>
   <joint
-    name="camera_color_joint"
+    name="camera_color_frame"
     type="fixed">
     <origin
@@ -298,5 +298,5 @@
   </link>
   <joint
-    name="camera_color_optical_joint"
+    name="camera_color_optical_frame"
     type="fixed">
     <origin
@@ -351,5 +351,5 @@
   </link>
   <joint
-    name="camera_depth_joint"
+    name="camera_depth_frame"
     type="fixed">
     <origin
@@ -404,5 +404,5 @@
   </link>
   <joint
-    name="camera_depth_optical_joint"
+    name="camera_depth_optical_frame"
     type="fixed">
     <origin

File: src/OrbbecSDK/orbbec_description/urdf/gemini2.urdf.xacro (robot description, xacro)
@@ -86,5 +86,5 @@
   </link>
   <joint
-    name="camera_botter_screw_joint"
+    name="camera_botter_screw_frame"
     type="fixed">
     <origin
@@ -139,5 +139,5 @@
   </link>
   <joint
-    name="camera_right_ir_joint"
+    name="camera_right_ir_frame"
     type="fixed">
     <origin
@@ -192,5 +192,5 @@
   </link>
   <joint
-    name="camera_right_ir_optical_joint"
+    name="camera_right_ir_optical_frame"
     type="fixed">
     <origin
@@ -245,5 +245,5 @@
   </link>
   <joint
-    name="camera_color_joint"
+    name="camera_color_frame"
     type="fixed">
     <origin
@@ -298,5 +298,5 @@
   </link>
   <joint
-    name="camera_color_optical_joint"
+    name="camera_color_optical_frame"
     type="fixed">
     <origin
@@ -351,5 +351,5 @@
   </link>
   <joint
-    name="camera_left_ir_joint"
+    name="camera_left_ir_frame"
     type="fixed">
     <origin
@@ -404,5 +404,5 @@
   </link>
   <joint
-    name="camera_left_ir_optical_joint"
+    name="camera_left_ir_optical_frame"
     type="fixed">
     <origin
@@ -457,5 +457,5 @@
   </link>
   <joint
-    name="camera_depth_joint"
+    name="camera_depth_frame"
     type="fixed">
     <origin

File: src/OrbbecSDK/orbbec_description/urdf/gemini2L.urdf.xacro (robot description, xacro)
@@ -86,5 +86,5 @@
   </link>
   <joint
-    name="camera_bottom_screw_joint"
+    name="camera_bottom_screw_frame"
     type="fixed">
     <origin
@@ -139,5 +139,5 @@
   </link>
   <joint
-    name="camera_right_ir_joint"
+    name="camera_right_ir_frame"
     type="fixed">
     <origin
@@ -192,5 +192,5 @@
   </link>
   <joint
-    name="camera_right_ir_optical_joint"
+    name="camera_right_ir_optical_frame"
     type="fixed">
     <origin
@@ -245,5 +245,5 @@
   </link>
   <joint
-    name="camera_left_ir_joint"
+    name="camera_left_ir_frame"
     type="fixed">
     <origin
@@ -298,5 +298,5 @@
   </link>
   <joint
-    name="camera_left_ir_optical_joint"
+    name="camera_left_ir_optical_frame"
     type="fixed">
     <origin
@@ -351,5 +351,5 @@
   </link>
   <joint
-    name="camera_color_joint"
+    name="camera_color_frame"
     type="fixed">
     <origin
@@ -404,5 +404,5 @@
   </link>
   <joint
-    name="camera_color_optical_joint"
+    name="camera_color_optical_frame"
     type="fixed">
     <origin
@@ -457,5 +457,5 @@
   </link>
   <joint
-    name="camera_imu_joint"
+    name="camera_imu_frame"
     type="fixed">
     <origin
@@ -510,5 +510,5 @@
   </link>
   <joint
-    name="camera_depth_joint"
+    name="camera_depth_frame"
     type="fixed">
     <origin

File: src/OrbbecSDK/orbbec_description/urdf/gemini335L_336L.urdf.xacro (robot description, xacro)
@@ -86,5 +86,5 @@
   </link>
   <joint
-    name="camera_color_screw_joint"
+    name="camera_color_screw_frame"
     type="fixed">
     <origin
@@ -139,5 +139,5 @@
   </link>
   <joint
-    name="camera_IMU_joint"
+    name="camera_IMU_frame"
     type="fixed">
     <origin
@@ -192,5 +192,5 @@
   </link>
   <joint
-    name="camera_depth_joint"
+    name="camera_depth_frame"
     type="fixed">
     <origin
@@ -245,5 +245,5 @@
   </link>
   <joint
-    name="camera_left_ir_joint"
+    name="camera_left_ir_frame"
     type="fixed">
     <origin
@@ -298,5 +298,5 @@
   </link>
   <joint
-    name="camera_left_ir_optical_joint"
+    name="camera_left_ir_optical_frame"
     type="fixed">
     <origin
@@ -351,5 +351,5 @@
   </link>
   <joint
-    name="camera_right_ir_joint"
+    name="camera_right_ir_frame"
     type="fixed">
     <origin
@@ -404,5 +404,5 @@
   </link>
   <joint
-    name="camera_right_ir_optical_joint"
+    name="camera_right_ir_optical_frame"
     type="fixed">
     <origin
@@ -457,5 +457,5 @@
   </link>
   <joint
-    name="camera_color_joint"
+    name="camera_color_frame"
     type="fixed">
     <origin
@@ -510,5 +510,5 @@
   </link>
   <joint
-    name="camera_color_optical_joint"
+    name="camera_color_optical_frame"
     type="fixed">
     <origin

File: src/duojin01_description/urdf/duojin01.xacro (robot description, xacro)
@@ -10,4 +10,5 @@
   <xacro:property name="use_shaft_collision" value="false" />
   <xacro:include filename="sensors/lidar.xacro" />
+  <xacro:include filename="sensors/camera.xacro" />
   <xacro:macro name="box_inertial" params="m x y z">
     <inertial>
@@ -209,4 +210,31 @@
     </inertial>
   </link>
+  <link name="depth_cam">
+    <visual>
+      <origin xyz="0 0 0.0" rpy="0 0 0" />
+      <geometry>
+        <mesh filename="package://duojin01_description/meshes/depth_camera.stl"
+          scale="1 1 1" />
+      </geometry>
+      <material name="black" />
+    </visual>
+  </link>
+  <joint name="depth_cam_joint" type="fixed">
+    <origin xyz="0.15 0 0.1" rpy="0 0 0" />
+    <parent link="base_link" />
+    <child link="depth_cam" />
+  </joint>
+  <!-- Simulated RGBD camera attached on depth_cam link -->
+  <xacro:rgbd_camera_sensor
+    reference_link="depth_cam"
+    sensor_name="depth_cam_rgbd"
+    topic="/camera"
+    update_rate="15"
+    hfov="1.047"
+    width="640"
+    height="480"
+    near_clip="0.1"
+    far_clip="10.0"
+    visualize="false" />
   <gazebo>
     <!-- 监听 ROS Topic /cmd_vel,用来直接驱动车辆全向移动 -->
