Commit message: fix(x11): improve stability and performance

File: src/duojin01_description/urdf/duojin01.xacro (robot description, xacro)
@@ -9,4 +9,11 @@
   <xacro:property name="wheel_mu2" value="$(optenv DUOJIN01_WHEEL_MU2 0.0)" />
   <xacro:property name="use_shaft_collision" value="false" />
+  <xacro:property name="sim_camera_enabled" value="$(optenv DUOJIN01_SIM_CAMERA_ENABLED true)" />
+  <xacro:property name="sim_camera_update_rate" value="$(optenv DUOJIN01_SIM_CAMERA_UPDATE_RATE 15)" />
+  <xacro:property name="sim_camera_hfov" value="$(optenv DUOJIN01_SIM_CAMERA_HFOV 1.047)" />
+  <xacro:property name="sim_camera_width" value="$(optenv DUOJIN01_SIM_CAMERA_WIDTH 640)" />
+  <xacro:property name="sim_camera_height" value="$(optenv DUOJIN01_SIM_CAMERA_HEIGHT 480)" />
+  <xacro:property name="sim_camera_near_clip" value="$(optenv DUOJIN01_SIM_CAMERA_NEAR_CLIP 0.1)" />
+  <xacro:property name="sim_camera_far_clip" value="$(optenv DUOJIN01_SIM_CAMERA_FAR_CLIP 10.0)" />
   <xacro:include filename="sensors/lidar.xacro" />
   <xacro:include filename="sensors/camera.xacro" />
@@ -225,16 +232,18 @@
     <child link="depth_cam" />
   </joint>
-  <!-- Simulated RGBD camera attached on depth_cam link -->
-  <xacro:rgbd_camera_sensor
-    reference_link="depth_cam"
-    sensor_name="depth_cam_rgbd"
-    topic="/camera"
-    update_rate="15"
-    hfov="1.047"
-    width="640"
-    height="480"
-    near_clip="0.1"
-    far_clip="10.0"
-    visualize="false" />
+  <xacro:if value="${str(sim_camera_enabled).lower() == 'true' or str(sim_camera_enabled) == '1'}">
+    <!-- Simulated RGBD camera attached on depth_cam link -->
+    <xacro:rgbd_camera_sensor
+      reference_link="depth_cam"
+      sensor_name="depth_cam_rgbd"
+      topic="/camera"
+      update_rate="${sim_camera_update_rate}"
+      hfov="${sim_camera_hfov}"
+      width="${sim_camera_width}"
+      height="${sim_camera_height}"
+      near_clip="${sim_camera_near_clip}"
+      far_clip="${sim_camera_far_clip}"
+      visualize="false" />
+  </xacro:if>
   <gazebo>
     <!-- 监听 ROS Topic /cmd_vel,用来直接驱动车辆全向移动 -->

Commit message: migrate to gz-sim Harmonic; drop Ignition; polish sim details

File: src/duojin01_description/urdf/duojin01.xacro (robot description, xacro)
@@ -1,11 +1,13 @@
 <?xml version="1.0"?>
 <robot name="duojin01" xmlns:xacro="http://ros.org/wiki/xacro">
-  <!-- 该 URDF 仅适用于 Gazebo Ignition -->
+  <!-- 该 URDF 仅适用于 Gazebo Harmonic (gz-sim) -->
   <xacro:property name="PI" value="3.1415926535897931" />
   <xacro:property name="wheel_radius" value="0.050" />
   <xacro:property name="wheel_width" value="0.0505" />
-  <!-- 摩擦为 0 ，故轮仅产生视觉效果，不参与车辆的实际驱动 -->
-  <xacro:property name="wheel_mu1" value="$(optenv DUOJIN01_WHEEL_MU1 0.0)" />
-  <xacro:property name="wheel_mu2" value="$(optenv DUOJIN01_WHEEL_MU2 0.0)" />
+  <!-- Default sim dynamics: use direct body velocity control so Nav2 omni commands (vx, vy, wz) are faithfully applied in sim -->
+  <xacro:property name="wheel_mu1" value="$(optenv DUOJIN01_WHEEL_MU1 2.0)" />
+  <xacro:property name="wheel_mu2" value="$(optenv DUOJIN01_WHEEL_MU2 2.0)" />
+  <xacro:property name="sim_velocity_control_enabled" value="$(optenv DUOJIN01_SIM_VELOCITY_CONTROL_ENABLED true)" />
+  <xacro:property name="sim_mecanum_visual_drive_enabled" value="$(optenv DUOJIN01_SIM_MECANUM_VISUAL_DRIVE_ENABLED false)" />
   <xacro:property name="use_shaft_collision" value="false" />
   <xacro:property name="sim_camera_enabled" value="$(optenv DUOJIN01_SIM_CAMERA_ENABLED true)" />
@@ -247,12 +249,14 @@
   </xacro:if>
   <gazebo>
-    <!-- 监听 ROS Topic /cmd_vel,用来直接驱动车辆全向移动 -->
-    <plugin filename="ignition-gazebo-velocity-control-system"
-      name="ignition::gazebo::systems::VelocityControl">
-      <topic>/cmd_vel</topic>
-    </plugin>
+    <xacro:if value="${str(sim_velocity_control_enabled).lower() == 'true' or str(sim_velocity_control_enabled) == '1'}">
+      <!-- Listen /cmd_vel and directly apply body velocity in simulation -->
+      <plugin filename="gz-sim-velocity-control-system"
+        name="gz::sim::systems::VelocityControl">
+        <topic>/cmd_vel</topic>
+      </plugin>
+    </xacro:if>
     <!-- 计算并发布机器人相对于 odom_frame 的坐标 -->
-    <plugin filename="ignition-gazebo-odometry-publisher-system"
-      name="ignition::gazebo::systems::OdometryPublisher">
+    <plugin filename="gz-sim-odometry-publisher-system"
+      name="gz::sim::systems::OdometryPublisher">
       <odom_frame>odom</odom_frame>
       <robot_base_frame>base_footprint</robot_base_frame>
@@ -261,20 +265,21 @@
       <odom_topic>/sim/odom</odom_topic>
     </plugin>
-    <!-- 监听 ROS Topic
-    /cmd_vel,将速度分配到四个轮子；为了提高性能，本仿真为使用真实的、每个滚子可动的麦轮，无法通过该插件实现全向移动，故目前该插件仅用于实现车轮转动的视觉效果 -->
-    <plugin filename="ignition-gazebo-mecanum-drive-system"
-      name="ignition::gazebo::systems::MecanumDrive">
-      <front_left_joint>upper_left_wheel_joint</front_left_joint>
-      <front_right_joint>upper_right_wheel_joint</front_right_joint>
-      <back_left_joint>lower_left_wheel_joint</back_left_joint>
-      <back_right_joint>lower_right_wheel_joint</back_right_joint>
-      <wheel_separation>0.208</wheel_separation>
-      <wheelbase>0.325</wheelbase>
-      <wheel_radius>${wheel_radius}</wheel_radius>
-      <topic>/cmd_vel</topic>
-    </plugin>
+    <xacro:if value="${str(sim_mecanum_visual_drive_enabled).lower() == 'true' or str(sim_mecanum_visual_drive_enabled) == '1'}">
+      <!-- Optional physically-driven mecanum plugin. Keep disabled by default to avoid cmd_vel double-control with VelocityControl. -->
+      <plugin filename="gz-sim-mecanum-drive-system"
+        name="gz::sim::systems::MecanumDrive">
+        <front_left_joint>upper_left_wheel_joint</front_left_joint>
+        <front_right_joint>upper_right_wheel_joint</front_right_joint>
+        <back_left_joint>lower_left_wheel_joint</back_left_joint>
+        <back_right_joint>lower_right_wheel_joint</back_right_joint>
+        <wheel_separation>0.208</wheel_separation>
+        <wheelbase>0.325</wheelbase>
+        <wheel_radius>${wheel_radius}</wheel_radius>
+        <topic>/cmd_vel</topic>
+      </plugin>
+    </xacro:if>
     <!-- 发布每个轮子当前转动的角度和速度 -->
-    <plugin filename="ignition-gazebo-joint-state-publisher-system"
-      name="ignition::gazebo::systems::JointStatePublisher">
+    <plugin filename="gz-sim-joint-state-publisher-system"
+      name="gz::sim::systems::JointStatePublisher">
       <topic>/joint_states</topic>
     </plugin>

File: src/duojin01_description/urdf/sensors/lidar.xacro (robot description, xacro)
@@ -77,5 +77,5 @@
           </range>
         </lidar>
-        <alwaysOn>1</alwaysOn>
+        <always_on>1</always_on>
         <visualize>false</visualize>
       </sensor>

Commit message: update URDF

File: src/duojin01_description/urdf/duojin01.xacro (robot description, xacro)
@@ -1,287 +1,5 @@
 <?xml version="1.0"?>
 <robot name="duojin01" xmlns:xacro="http://ros.org/wiki/xacro">
-  <!-- 该 URDF 仅适用于 Gazebo Harmonic (gz-sim) -->
-  <xacro:property name="PI" value="3.1415926535897931" />
-  <xacro:property name="wheel_radius" value="0.050" />
-  <xacro:property name="wheel_width" value="0.0505" />
-  <!-- Default sim dynamics: use direct body velocity control so Nav2 omni commands (vx, vy, wz) are faithfully applied in sim -->
-  <xacro:property name="wheel_mu1" value="$(optenv DUOJIN01_WHEEL_MU1 2.0)" />
-  <xacro:property name="wheel_mu2" value="$(optenv DUOJIN01_WHEEL_MU2 2.0)" />
-  <xacro:property name="sim_velocity_control_enabled" value="$(optenv DUOJIN01_SIM_VELOCITY_CONTROL_ENABLED true)" />
-  <xacro:property name="sim_mecanum_visual_drive_enabled" value="$(optenv DUOJIN01_SIM_MECANUM_VISUAL_DRIVE_ENABLED false)" />
-  <xacro:property name="use_shaft_collision" value="false" />
-  <xacro:property name="sim_camera_enabled" value="$(optenv DUOJIN01_SIM_CAMERA_ENABLED true)" />
-  <xacro:property name="sim_camera_update_rate" value="$(optenv DUOJIN01_SIM_CAMERA_UPDATE_RATE 15)" />
-  <xacro:property name="sim_camera_hfov" value="$(optenv DUOJIN01_SIM_CAMERA_HFOV 1.047)" />
-  <xacro:property name="sim_camera_width" value="$(optenv DUOJIN01_SIM_CAMERA_WIDTH 640)" />
-  <xacro:property name="sim_camera_height" value="$(optenv DUOJIN01_SIM_CAMERA_HEIGHT 480)" />
-  <xacro:property name="sim_camera_near_clip" value="$(optenv DUOJIN01_SIM_CAMERA_NEAR_CLIP 0.1)" />
-  <xacro:property name="sim_camera_far_clip" value="$(optenv DUOJIN01_SIM_CAMERA_FAR_CLIP 10.0)" />
-  <xacro:include filename="sensors/lidar.xacro" />
-  <xacro:include filename="sensors/camera.xacro" />
-  <xacro:macro name="box_inertial" params="m x y z">
-    <inertial>
-      <mass value="${m}" />
-      <inertia
-        ixx="${m*(y*y+z*z)/12}" ixy="0" ixz="0"
-        iyy="${m*(x*x+z*z)/12}" iyz="0"
-        izz="${m*(x*x+y*y)/12}" />
-    </inertial>
-  </xacro:macro>
-  <xacro:macro name="cylinder_inertial" params="m r h">
-    <inertial>
-      <mass value="${m}" />
-      <inertia
-        ixx="${m*(3*r*r+h*h)/12}" ixy="0" ixz="0"
-        iyy="${m*(3*r*r+h*h)/12}" iyz="0"
-        izz="${m*r*r/2}" />
-    </inertial>
-  </xacro:macro>
-  <material name="black">
-    <color rgba="0.15 0.15 0.15 1.0" />
-  </material>
-  <material name="light_grey">
-    <color rgba="0.4 0.4 0.4 1.0" />
-  </material>
-  <material name="white">
-    <color rgba="1.0 1.0 1.0 1.0" />
-  </material>
-  <link name="base_footprint">
-  </link>
-  <joint name="base_link_joint" type="fixed">
-    <origin xyz="0 0 0" rpy="0 0 0" />
-    <parent link="base_footprint" />
-    <child link="base_link" />
-  </joint>
-  <link name="base_link">
-    <visual>
-      <origin xyz="0 0 0.02" rpy="0 0 0" />
-      <geometry>
-        <mesh filename="package://duojin01_description/meshes/base_visual.stl"
-          scale="0.001 0.001 0.001" />
-      </geometry>
-      <material name="light_grey" />
-    </visual>
-    <visual name="surface_visual">
-      <origin xyz="0 0 0.14" rpy="0 0 0" />
-      <geometry>
-        <mesh filename="package://duojin01_description/meshes/surface_visual.stl"
-          scale="0.001 0.001 0.001" />
-      </geometry>
-      <material name="white" />
-    </visual>
-    <xacro:box_inertial m="10.0" x="0.4" y="0.3" z="0.1" />
-  </link>
-  <gazebo reference="base_link">
-    <material>Gazebo/Grey</material>
-  </gazebo>
-  <xacro:macro name="mecanum_wheel_unit"
-    params="prefix location_x location_y shaft_rpy wheel_mesh_file axis_sign">
-    <joint name="${prefix}_wheel_shaft_joint" type="fixed">
-      <origin xyz="${location_x} ${location_y} ${wheel_radius}" rpy="${shaft_rpy}" />
-      <parent link="base_link" />
-      <child link="${prefix}_wheel_shaft" />
-    </joint>
-    <link name="${prefix}_wheel_shaft">
-      <visual>
-        <geometry>
-          <mesh filename="package://duojin01_description/meshes/wheel_shaft.stl"
-            scale="0.001 0.001 0.001" />
-        </geometry>
-        <material name="black" />
-      </visual>
-      <xacro:if value="${use_shaft_collision}">
-        <collision>
-          <geometry>
-            <mesh filename="package://duojin01_description/meshes/wheel_shaft.stl"
-              scale="0.001 0.001 0.001" />
-          </geometry>
-        </collision>
-      </xacro:if>
-      <xacro:box_inertial m="0.2" x="0.05" y="0.05" z="0.05" />
-    </link>
-    <joint name="${prefix}_wheel_joint" type="continuous">
-      <origin xyz="0 0.042 0" rpy="0 0 0" />
-      <parent link="${prefix}_wheel_shaft" />
-      <child link="${prefix}_wheel" />
-      <axis xyz="0 ${axis_sign} 0" />
-    </joint>
-    <link name="${prefix}_wheel">
-      <visual>
-        <geometry>
-          <mesh filename="${wheel_mesh_file}" scale="0.001 0.001 0.001" />
-        </geometry>
-        <material name="black" />
-      </visual>
-      <collision name="${prefix}_wheel_collision">
-        <origin xyz="0 0 0" rpy="${PI/2} 0 0" />
-        <geometry>
-          <cylinder radius="${wheel_radius}" length="${wheel_width}" />
-        </geometry>
-      </collision>
-      <xacro:cylinder_inertial m="0.5" r="${wheel_radius}" h="${wheel_width}" />
-    </link>
-    <gazebo reference="${prefix}_wheel">
-      <material>Gazebo/Black</material>
-      <collision name="${prefix}_wheel_collision">
-        <surface>
-          <friction>
-            <ode>
-              <mu>${wheel_mu1}</mu>
-              <mu2>${wheel_mu2}</mu2>
-            </ode>
-          </friction>
-        </surface>
-      </collision>
-    </gazebo>
-  </xacro:macro>
-  <xacro:mecanum_wheel_unit
-    prefix="upper_left"
-    location_x="0.175" location_y="0.104"
-    shaft_rpy="0 0 0"
-    wheel_mesh_file="package://duojin01_description/meshes/mecanum_wheel_left.stl"
-    axis_sign="-1" />
-  <xacro:mecanum_wheel_unit
-    prefix="lower_left"
-    location_x="-0.150" location_y="0.104"
-    shaft_rpy="0 0 0"
-    wheel_mesh_file="package://duojin01_description/meshes/mecanum_wheel_right.stl"
-    axis_sign="-1" />
-  <xacro:mecanum_wheel_unit
-    prefix="upper_right"
-    location_x="0.175" location_y="-0.104"
-    shaft_rpy="${PI} 0 0"
-    wheel_mesh_file="package://duojin01_description/meshes/mecanum_wheel_right.stl"
-    axis_sign="1" />
-  <xacro:mecanum_wheel_unit
-    prefix="lower_right"
-    location_x="-0.150" location_y="-0.104"
-    shaft_rpy="${PI} 0 0"
-    wheel_mesh_file="package://duojin01_description/meshes/mecanum_wheel_left.stl"
-    axis_sign="1" />
-  <xacro:macro name="pillar" params="prefix x y">
-    <joint name="${prefix}_pillar_joint" type="fixed">
-      <origin xyz="${x} ${y} 0.098" rpy="0 0 0" />
-      <parent link="base_link" />
-      <child link="${prefix}_pillar" />
-    </joint>
-    <link name="${prefix}_pillar">
-      <visual>
-        <geometry>
-          <box size="0.015 0.015 0.10" />
-        </geometry>
-        <material name="light_grey" />
-      </visual>
-      <collision>
-        <geometry>
-          <box size="0.015 0.015 0.10" />
-        </geometry>
-      </collision>
-      <xacro:box_inertial m="0.05" x="0.015" y="0.015" z="0.1" />
-    </link>
-  </xacro:macro>
-  <xacro:pillar prefix="upper_left" x="0.175" y="0.100" />
-  <xacro:pillar prefix="lower_left" x="-0.165" y="0.100" />
-  <xacro:pillar prefix="upper_right" x="0.175" y="-0.100" />
-  <xacro:pillar prefix="lower_right" x="-0.145" y="-0.100" />
-  <joint name="computer_joint" type="fixed">
-    <origin xyz="0.135 0 0.175" rpy="0 0 0" />
-    <parent link="base_link" />
-    <child link="computer" />
-  </joint>
-  <link name="computer">
-    <visual>
-      <geometry>
-        <box size="0.13 0.13 0.05" />
-      </geometry>
-      <material name="black" />
-    </visual>
-    <collision>
-      <geometry>
-        <box size="0.13 0.13 0.05" />
-      </geometry>
-    </collision>
-    <xacro:box_inertial m="0.5" x="0.13" y="0.13" z="0.05" />
-  </link>
-  <xacro:lidar_sensor parent="base_link">
-    <origin xyz="0.1 0 0.11" rpy="0 0 0" />
-  </xacro:lidar_sensor>
-  <joint name="imu_joint" type="fixed">
-    <origin xyz="0 0 0" rpy="0 0 0" />
-    <parent link="base_link" />
-    <child link="imu_link" />
-  </joint>
-  <link name="imu_link">
-    <inertial>
-      <mass value="0.01" />
-      <origin xyz="0 0 0" />
-      <inertia ixx="1e-6" ixy="0" ixz="0" iyy="1e-6" iyz="0" izz="1e-6" />
-    </inertial>
-  </link>
-  <link name="depth_cam">
-    <visual>
-      <origin xyz="0 0 0.0" rpy="0 0 0" />
-      <geometry>
-        <mesh filename="package://duojin01_description/meshes/depth_camera.stl"
-          scale="1 1 1" />
-      </geometry>
-      <material name="black" />
-    </visual>
-  </link>
-  <joint name="depth_cam_joint" type="fixed">
-    <origin xyz="0.15 0 0.1" rpy="0 0 0" />
-    <parent link="base_link" />
-    <child link="depth_cam" />
-  </joint>
-  <xacro:if value="${str(sim_camera_enabled).lower() == 'true' or str(sim_camera_enabled) == '1'}">
-    <!-- Simulated RGBD camera attached on depth_cam link -->
-    <xacro:rgbd_camera_sensor
-      reference_link="depth_cam"
-      sensor_name="depth_cam_rgbd"
-      topic="/camera"
-      update_rate="${sim_camera_update_rate}"
-      hfov="${sim_camera_hfov}"
-      width="${sim_camera_width}"
-      height="${sim_camera_height}"
-      near_clip="${sim_camera_near_clip}"
-      far_clip="${sim_camera_far_clip}"
-      visualize="false" />
-  </xacro:if>
-  <gazebo>
-    <xacro:if value="${str(sim_velocity_control_enabled).lower() == 'true' or str(sim_velocity_control_enabled) == '1'}">
-      <!-- Listen /cmd_vel and directly apply body velocity in simulation -->
-      <plugin filename="gz-sim-velocity-control-system"
-        name="gz::sim::systems::VelocityControl">
-        <topic>/cmd_vel</topic>
-      </plugin>
-    </xacro:if>
-    <!-- 计算并发布机器人相对于 odom_frame 的坐标 -->
-    <plugin filename="gz-sim-odometry-publisher-system"
-      name="gz::sim::systems::OdometryPublisher">
-      <odom_frame>odom</odom_frame>
-      <robot_base_frame>base_footprint</robot_base_frame>
-      <dimensions>2</dimensions>
-      <odom_publish_frequency>200</odom_publish_frequency>
-      <odom_topic>/sim/odom</odom_topic>
-    </plugin>
-    <xacro:if value="${str(sim_mecanum_visual_drive_enabled).lower() == 'true' or str(sim_mecanum_visual_drive_enabled) == '1'}">
-      <!-- Optional physically-driven mecanum plugin. Keep disabled by default to avoid cmd_vel double-control with VelocityControl. -->
-      <plugin filename="gz-sim-mecanum-drive-system"
-        name="gz::sim::systems::MecanumDrive">
-        <front_left_joint>upper_left_wheel_joint</front_left_joint>
-        <front_right_joint>upper_right_wheel_joint</front_right_joint>
-        <back_left_joint>lower_left_wheel_joint</back_left_joint>
-        <back_right_joint>lower_right_wheel_joint</back_right_joint>
-        <wheel_separation>0.208</wheel_separation>
-        <wheelbase>0.325</wheelbase>
-        <wheel_radius>${wheel_radius}</wheel_radius>
-        <topic>/cmd_vel</topic>
-      </plugin>
-    </xacro:if>
-    <!-- 发布每个轮子当前转动的角度和速度 -->
-    <plugin filename="gz-sim-joint-state-publisher-system"
-      name="gz::sim::systems::JointStatePublisher">
-      <topic>/joint_states</topic>
-    </plugin>
-  </gazebo>
+  <xacro:include filename="duojin01_shared.xacro" />
+  <xacro:duojin01_shared_model use_shaft_collision="false" />
 </robot>
