Commit message: refactor: remove depth camera and safety modules
Keep the hardware workspace on Ubuntu 22.04 and ROS 2 Humble with 10 packages. Connect ordinary velocity arbitration directly to the base driver, remove obsolete launch and Docker dependencies, and document current modules and upstream lidar differences.

File: src/duojin01_description/urdf/duojin01_hardware.xacro (robot description, xacro)
@@ -223,19 +223,4 @@
       </inertial>
     </link>
-    <link name="depth_cam">
-      <visual>
-        <origin xyz="0 0 0.0" rpy="0 0 0" />
-        <geometry>
-          <mesh filename="package://duojin01_description/meshes/depth_camera.stl"
-            scale="1 1 1" />
-        </geometry>
-        <material name="black" />
-      </visual>
-    </link>
-    <joint name="depth_cam_joint" type="fixed">
-      <origin xyz="0.17 0 0.1" rpy="0 0 0" />
-      <parent link="base_link" />
-      <child link="depth_cam" />
-    </joint>
   </xacro:macro>
 </robot>
